File: freesoc/freesoc_1.1.sch (EAGLE design)
At the start: 86 parts, among them IC1 CY8C3X66AXI, IC2 CY7C68015A, IC4 24LC00OT, SW1 JS202011SCQN, Y2 ATS240C, Y3 AB26T-32.768KHZ, Y4 ATS240C

Commit message: Updates to boards for production
Parts:
- removed ANALOG, POWER: M20-7820642, pinhead:PINHD-1X6
- removed C26, C27: 10nF, SparkFun:CAP0402-CAP
- added JP11: (no value), SparkFun:M07
- added JP12: (no value), SparkFun:M06SIP
- C1, C10, C11, C12, C14, C15, C16, C17, C6, C7, C8, C9: PN (none) -> LMK105BJ104KV-F
- C13, C2, C23, C3: PN (none) -> C0805C106K4PACTU
- C18, C21, C29, C30: PN (none) -> GRM1555C1H180FZ01D
- C19, C20, C22, C24, C25: PN (none) -> JMK105BJ105KV-F
- C32, C33: PN (none) -> GRM1555C1H120FZ01D
- C4: PN (none) -> TMK105B7103KV-F
- C5: PN (none) -> CC0603KRX5R5BB225
- D1, D2, D3, D4, D5, D6: PN (none) -> PMEG3010ER
- IC1: PN (none) -> CY8C5568AXI-060
- IC2: PN (none) -> CY7C68013A-56LTXC
- IC4: PN (none) -> 24LC00T
- JP1, JP2, JP3, JP4, JP5: device SparkFun:M05X2RAF -> SparkFun:M05X2BLANK
- JP6: PN (none) -> S2B-PH-SM4-TB
- LED1, LED2, LED5: PN (none) -> VLMW1300-GS08
- R1, R3: PN (none) -> RR0510P-104-D
- R10: PN (none) -> ERJ-2RKF3601X
- R11, R12, R15, R9: PN (none) -> ERJ-2RKF2201X
- R18, R7, R8: PN (none) -> CRCW0603150RFKEA
- R2: PN (none) -> ERJ-2GEJ103X
- R4: value 6.6k -> 6.49k; PN (none) -> CRCW04026R49FKED
- R5, R6: PN (none) -> ERA-6AHD220V
- REG3V3, REG5V0: PN (none) -> NCP5500DADJR2G
- S2: PN (none) -> TL1105F160Q
- SW1: PN (none) -> JS202011SCQN
- U$5, U$6: PN (none) -> 10033526-N3212LF
- Y2, Y4: PN (none) -> ATS240C
- Y3: PN (none) -> AB26T-32.768KHZ
- Z1, Z2, Z3, Z4, Z5, Z6: PN (none) -> CG0603MLC-05LE
Connections:
- net !XRES: now also JP11.6; no longer POWER.1
- net 5V: now also JP11.4; no longer POWER.3
- net GND: now also JP11.2, JP11.3; no longer C26.2, C27.2, POWER.4, POWER.5
- net N$13: no longer C27.1
- net N$25: no longer C26.1
- net P16: now also JP12.1; no longer ANALOG.1
- net P17: now also JP12.2; no longer ANALOG.2
- net P54: now also JP12.3; no longer ANALOG.3
- net P55: now also JP12.4; no longer ANALOG.4
- net P56: now also JP12.5; no longer ANALOG.5
- net P57: now also JP12.6; no longer ANALOG.6
- net VDD: now also JP11.5; no longer POWER.2
- net VIN: now also JP11.1; no longer POWER.6
- net VPSOC: now also JP11.7
