File: freesoc mini/freesoc_mini_1.0.sch (EAGLE design)
At the start: 50 parts, among them IC1 CY7C68013A-56QFNLFXC, IC2 24LC00OT, Y1 XRCGB24M000F0L00R0

Commit message: Updates to boards for production
Parts:
- removed R3, R4, R5: NOLOAD, SparkFun:RESISTOR0402-RES
- C1, C10, C11, C13, C15, C21, C22, C23, C24, C25, C27, C3, C4, C7, C8: PN (none) -> LMK105BJ104KV-F
- C12, C14, C29, C31, C5, C6, C9: PN (none) -> JMK105BJ105KV-F
- C16, C17: PN (none) -> CC0603KRX5R6BB475
- C19, C20: PN (none) -> GJM1555C1H100FB01D
- C2: PN (none) -> JMK105BJ225MV-F
- C26, C28: PN (none) -> TMK105B7103KV-F
- D1, D2: PN (none) -> NSVR0320MW2T1G
- IC1: PN (none) -> CY7C68013A-56LTXC
- IC2: PN (none) -> 24LC00T
- R10, R11: PN (none) -> ERJ-2RKF2201X
- R12, R9: PN (none) -> RR0510P-104-D
- R13: PN (none) -> ERJ-2RKF1001X
- R8: PN (none) -> ERJ-2GEJ103X
- U$1: PN (none) -> CY8C5568LTI-114
- U$3: PN (none) -> FAN2558S36X
- USB-MINIB: PN (none) -> 10033526-N3212LF
- Y1: PN (none) -> XRCGB24M000F0L00R0
Connections:
- net SWDCK: no longer R4.1
- net SWDIO: no longer R3.1
- net SWV: no longer R5.1
- net VCC: no longer R3.2, R4.2, R5.2
